Commit message: Update PROBOT Anno demos

File: probot_description/urdf/probot_anno.xacro (robot description, xacro)
@@ -11,6 +11,6 @@
     <inertial>
       <origin xyz="-0.010934 0.23134 0.0051509" rpy="0 0 0" />
-      <mass value="19.574" />
-      <inertia ixx="0" ixy="0" ixz="0" iyy="0" iyz="0" izz="0" />
+      <mass value="0.00001" />
+      <inertia ixx="10" ixy="0.0" ixz="0.0" iyy="10" iyz="0.0" izz="10" />
     </inertial>
     <visual>
@@ -33,6 +33,6 @@
     <inertial>
       <origin xyz="-0.010934 0.23134 0.0051509" rpy="0 0 0" />
-      <mass value="19.574" />
-      <inertia ixx="0" ixy="0" ixz="0" iyy="0" iyz="0" izz="0" />
+      <mass value="0.00001" />
+      <inertia ixx="10" ixy="0.0" ixz="0.0" iyy="10" iyz="0.0" izz="10" />
     </inertial>
     <visual>
@@ -62,6 +62,6 @@
     <inertial>
       <origin xyz="-0.010934 0.23134 0.0051509" rpy="0 0 0" />
-      <mass value="19.574" />
-      <inertia ixx="0" ixy="0" ixz="0" iyy="0" iyz="0" izz="0" />
+      <mass value="0.00001" />
+      <inertia ixx="10" ixy="0.0" ixz="0.0" iyy="10" iyz="0.0" izz="10" />
     </inertial>
     <visual>
@@ -91,6 +91,6 @@
     <inertial>
       <origin xyz="-0.010934 0.23134 0.0051509" rpy="0 0 0" />
-      <mass value="19.574" />
-      <inertia ixx="0" ixy="0" ixz="0" iyy="0" iyz="0" izz="0" />
+      <mass value="0.00001" />
+      <inertia ixx="10" ixy="0.0" ixz="0.0" iyy="10" iyz="0.0" izz="10" />
     </inertial>
     <visual>
@@ -120,6 +120,6 @@
     <inertial>
       <origin xyz="-0.010934 0.23134 0.0051509" rpy="0 0 0" />
-      <mass value="19.574" />
-      <inertia ixx="0" ixy="0" ixz="0" iyy="0" iyz="0" izz="0" />
+      <mass value="0.00001" />
+      <inertia ixx="10" ixy="0.0" ixz="0.0" iyy="10" iyz="0.0" izz="10" />
     </inertial>
     <visual>
@@ -149,6 +149,6 @@
     <inertial>
       <origin xyz="-0.010934 0.23134 0.0051509" rpy="0 0 0" />
-      <mass value="19.574" />
-      <inertia ixx="0" ixy="0" ixz="0" iyy="0" iyz="0" izz="0" />
+      <mass value="0.00001" />
+      <inertia ixx="10" ixy="0.0" ixz="0.0" iyy="10" iyz="0.0" izz="10" />
     </inertial>
     <visual>
@@ -178,6 +178,6 @@
     <inertial>
       <origin xyz="-0.010934 0.23134 0.0051509" rpy="0 0 0" />
-      <mass value="19.574" />
-      <inertia ixx="0" ixy="0" ixz="0" iyy="0" iyz="0" izz="0" />
+      <mass value="0.00001" />
+      <inertia ixx="10" ixy="0.0" ixz="0.0" iyy="10" iyz="0.0" izz="10" />
     </inertial>
     <visual>

Commit message: Update robot software 1.1.0

File: probot_description/urdf/probot_anno.xacro (robot description, xacro)
@@ -4,5 +4,5 @@
   <link name="base_footprint"/>
   <joint name="joint_0" type="fixed">
-    <origin xyz="0 0 0.0532" rpy="0 0 0" />
+    <origin xyz="0 0 0.02" rpy="0 0 0" />
     <parent link="base_footprint" />
     <child link="base_link" />
@@ -15,5 +15,5 @@
     </inertial>
     <visual>
-      <origin xyz="0.017266 0 0" rpy="0 0 0" />
+      <origin xyz="0.017266 0 0.0315" rpy="0 0 0" />
       <geometry>
         <mesh filename="package://probot_description/meshes/base_link.STL" />
@@ -24,5 +24,5 @@
     </visual>
     <collision>
-      <origin xyz="0.017266 0 0" rpy="0 0 0" />
+      <origin xyz="0.017266 0 0.0315" rpy="0 0 0" />
       <geometry>
         <mesh filename="package://probot_description/meshes/base_link.STL" />
@@ -53,5 +53,5 @@
   </link>
   <joint name="joint_1" type="revolute">
-    <origin xyz="0 0 0" rpy="1.5708 0 0" />
+    <origin xyz="0 0 0.0315" rpy="1.5708 0 0" />
     <parent link="base_link" />
     <child link="link_1" />
@@ -140,5 +140,5 @@
   </link>
   <joint name="joint_4" type="revolute">
-    <origin xyz="0.021 0 0.002" rpy="0 0 0" />
+    <origin xyz="0.023 0 0.0" rpy="0 0 0" />
     <parent link="link_3" />
     <child link="link_4" />
@@ -169,5 +169,5 @@
   </link>
   <joint name="joint_5" type="revolute">
-    <origin xyz="0.20586 0 0" rpy="0 0 0" />
+    <origin xyz="0.20585535 0 0" rpy="0 0 0" />
     <parent link="link_4" />
     <child link="link_5" />
@@ -206,5 +206,5 @@
   <link name="tool0"/>
   <joint name="joint_tool0" type="fixed">
-    <origin xyz="0 -0.013 0" rpy="0 0 0" />
+    <origin xyz="0 -0.013 0" rpy="${M_PI/2} 0 0" />
     <parent link="link_6" />
     <child link="tool0" />

File: probot_description/urdf/probot_anno_with_gripper.xacro (robot description, xacro)
@@ -6,5 +6,5 @@
   <link name="base_footprint"/>
   <joint name="joint_0" type="fixed">
-    <origin xyz="0 0 0.0532" rpy="0 0 0" />
+    <origin xyz="0 0 0.02" rpy="0 0 0" />
     <parent link="base_footprint" />
     <child link="base_link" />
@@ -17,5 +17,5 @@
     </inertial>
     <visual>
-      <origin xyz="0.017266 0 0" rpy="0 0 0" />
+      <origin xyz="0.017266 0 0.0315" rpy="0 0 0" />
       <geometry>
         <mesh filename="package://probot_description/meshes/base_link.STL" />
@@ -26,5 +26,5 @@
     </visual>
     <collision>
-      <origin xyz="0.017266 0 0" rpy="0 0 0" />
+      <origin xyz="0.017266 0 0.0315" rpy="0 0 0" />
       <geometry>
         <mesh filename="package://probot_description/meshes/base_link.STL" />
@@ -55,5 +55,5 @@
   </link>
   <joint name="joint_1" type="revolute">
-    <origin xyz="0 0 0" rpy="1.5708 0 0" />
+    <origin xyz="0 0 0.0315" rpy="1.5708 0 0" />
     <parent link="base_link" />
     <child link="link_1" />
@@ -142,5 +142,5 @@
   </link>
   <joint name="joint_4" type="revolute">
-    <origin xyz="0.021 0 0.002" rpy="0 0 0" />
+    <origin xyz="0.023 0 0.0" rpy="0 0 0" />
     <parent link="link_3" />
     <child link="link_4" />
@@ -171,5 +171,5 @@
   </link>
   <joint name="joint_5" type="revolute">
-    <origin xyz="0.20586 0 0" rpy="0 0 0" />
+    <origin xyz="0.20585535 0 0" rpy="0 0 0" />
     <parent link="link_4" />
     <child link="link_5" />
@@ -208,10 +208,10 @@
   <link name="tool0"/>
   <joint name="joint_tool0" type="fixed">
-    <origin xyz="0 -0.02 0" rpy="0 0 0" />
+    <origin xyz="0 -0.013 0" rpy="${M_PI/2} 0 0" />
     <parent link="link_6" />
     <child link="tool0" />
   </joint>
    <!-- Attach the right gripper -->
-   <gripper parent="tool0" color="Green" xyz="0 -0.015 0.01" rpy="0 0 ${-M_PI/2}"/>
+   <gripper parent="tool0" color="Green" xyz="0 0.015 0.02" rpy="0 ${-M_PI/2} ${-M_PI/2}"/>
   <!-- Transmissions for ROS Control -->
   <xacro:macro name="transmission_block" params="joint_name">
