Commit message: Update robot software v2.0

File: probot_description/urdf/PROBOT_Anno/probot_anno.xacro (robot description, xacro)
@@ -17,5 +17,5 @@
       <origin xyz="0.017266 0 0.0315" rpy="0 0 0" />
       <geometry>
-        <mesh filename="package://probot_description/meshes/base_link.STL" />
+        <mesh filename="package://probot_description/meshes/PROBOT_Anno/base_link.STL" />
       </geometry>
       <material name="">
@@ -26,5 +26,5 @@
       <origin xyz="0.017266 0 0.0315" rpy="0 0 0" />
       <geometry>
-        <mesh filename="package://probot_description/meshes/base_link.STL" />
+        <mesh filename="package://probot_description/meshes/PROBOT_Anno/base_link.STL" />
       </geometry>
     </collision>
@@ -39,14 +39,14 @@
       <origin xyz="0 0 0" rpy="0 0 0" />
       <geometry>
-        <mesh filename="package://probot_description/meshes/link_1.STL" />
-      </geometry>
-      <material name="">
-        <color rgba="0.79216 0.81961 0.93333 1" />
-      </material>
-    </visual>
-    <collision>
-      <origin xyz="0 0 0" rpy="0 0 0" />
-      <geometry>
-        <mesh filename="package://probot_description/meshes/link_1.STL" />
+        <mesh filename="package://probot_description/meshes/PROBOT_Anno/link_1.STL" />
+      </geometry>
+      <material name="">
+        <color rgba="0.79216 0.81961 0.93333 1" />
+      </material>
+    </visual>
+    <collision>
+      <origin xyz="0 0 0" rpy="0 0 0" />
+      <geometry>
+        <mesh filename="package://probot_description/meshes/PROBOT_Anno/link_1.STL" />
       </geometry>
     </collision>
@@ -68,14 +68,14 @@
       <origin xyz="0 0 0" rpy="0 0 0" />
       <geometry>
-        <mesh filename="package://probot_description/meshes/link_2.STL" />
-      </geometry>
-      <material name="">
-        <color rgba="0.79216 0.81961 0.93333 1" />
-      </material>
-    </visual>
-    <collision>
-      <origin xyz="0 0 0" rpy="0 0 0" />
-      <geometry>
-        <mesh filename="package://probot_description/meshes/link_2.STL" />
+        <mesh filename="package://probot_description/meshes/PROBOT_Anno/link_2.STL" />
+      </geometry>
+      <material name="">
+        <color rgba="0.79216 0.81961 0.93333 1" />
+      </material>
+    </visual>
+    <collision>
+      <origin xyz="0 0 0" rpy="0 0 0" />
+      <geometry>
+        <mesh filename="package://probot_description/meshes/PROBOT_Anno/link_2.STL" />
       </geometry>
     </collision>
@@ -97,14 +97,14 @@
       <origin xyz="0 0 0" rpy="0 0 0" />
       <geometry>
-        <mesh filename="package://probot_description/meshes/link_3.STL" />
-      </geometry>
-      <material name="">
-        <color rgba="0.79216 0.81961 0.93333 1" />
-      </material>
-    </visual>
-    <collision>
-      <origin xyz="0 0 0" rpy="0 0 0" />
-      <geometry>
-        <mesh filename="package://probot_description/meshes/link_3.STL" />
+        <mesh filename="package://probot_description/meshes/PROBOT_Anno/link_3.STL" />
+      </geometry>
+      <material name="">
+        <color rgba="0.79216 0.81961 0.93333 1" />
+      </material>
+    </visual>
+    <collision>
+      <origin xyz="0 0 0" rpy="0 0 0" />
+      <geometry>
+        <mesh filename="package://probot_description/meshes/PROBOT_Anno/link_3.STL" />
       </geometry>
     </collision>
@@ -126,14 +126,14 @@
       <origin xyz="0 0 0" rpy="0 0 0" />
       <geometry>
-        <mesh filename="package://probot_description/meshes/link_4.STL" />
-      </geometry>
-      <material name="">
-        <color rgba="0.79216 0.81961 0.93333 1" />
-      </material>
-    </visual>
-    <collision>
-      <origin xyz="0 0 0" rpy="0 0 0" />
-      <geometry>
-        <mesh filename="package://probot_description/meshes/link_4.STL" />
+        <mesh filename="package://probot_description/meshes/PROBOT_Anno/link_4.STL" />
+      </geometry>
+      <material name="">
+        <color rgba="0.79216 0.81961 0.93333 1" />
+      </material>
+    </visual>
+    <collision>
+      <origin xyz="0 0 0" rpy="0 0 0" />
+      <geometry>
+        <mesh filename="package://probot_description/meshes/PROBOT_Anno/link_4.STL" />
       </geometry>
     </collision>
@@ -155,14 +155,14 @@
       <origin xyz="0 0 0" rpy="0 0 0" />
       <geometry>
-        <mesh filename="package://probot_description/meshes/link_5.STL" />
-      </geometry>
-      <material name="">
-        <color rgba="0.79216 0.81961 0.93333 1" />
-      </material>
-    </visual>
-    <collision>
-      <origin xyz="0 0 0" rpy="0 0 0" />
-      <geometry>
-        <mesh filename="package://probot_description/meshes/link_5.STL" />
+        <mesh filename="package://probot_description/meshes/PROBOT_Anno/link_5.STL" />
+      </geometry>
+      <material name="">
+        <color rgba="0.79216 0.81961 0.93333 1" />
+      </material>
+    </visual>
+    <collision>
+      <origin xyz="0 0 0" rpy="0 0 0" />
+      <geometry>
+        <mesh filename="package://probot_description/meshes/PROBOT_Anno/link_5.STL" />
       </geometry>
     </collision>
@@ -184,14 +184,14 @@
       <origin xyz="0 0 0" rpy="0 0 0" />
       <geometry>
-        <mesh filename="package://probot_description/meshes/link_6.STL" />
-      </geometry>
-      <material name="">
-        <color rgba="0.79216 0.81961 0.93333 1" />
-      </material>
-    </visual>
-    <collision>
-      <origin xyz="0 0 0" rpy="0 0 0" />
-      <geometry>
-        <mesh filename="package://probot_description/meshes/link_6.STL" />
+        <mesh filename="package://probot_description/meshes/PROBOT_Anno/link_6.STL" />
+      </geometry>
+      <material name="">
+        <color rgba="0.79216 0.81961 0.93333 1" />
+      </material>
+    </visual>
+    <collision>
+      <origin xyz="0 0 0" rpy="0 0 0" />
+      <geometry>
+        <mesh filename="package://probot_description/meshes/PROBOT_Anno/link_6.STL" />
       </geometry>
     </collision>

File: probot_description/urdf/PROBOT_Anno/probot_anno_with_gripper.xacro (robot description, xacro)
@@ -19,5 +19,5 @@
       <origin xyz="0.017266 0 0.0315" rpy="0 0 0" />
       <geometry>
-        <mesh filename="package://probot_description/meshes/base_link.STL" />
+        <mesh filename="package://probot_description/meshes/PROBOT_Anno/base_link.STL" />
       </geometry>
       <material name="">
@@ -28,5 +28,5 @@
       <origin xyz="0.017266 0 0.0315" rpy="0 0 0" />
       <geometry>
-        <mesh filename="package://probot_description/meshes/base_link.STL" />
+        <mesh filename="package://probot_description/meshes/PROBOT_Anno/base_link.STL" />
       </geometry>
     </collision>
@@ -41,14 +41,14 @@
       <origin xyz="0 0 0" rpy="0 0 0" />
       <geometry>
-        <mesh filename="package://probot_description/meshes/link_1.STL" />
-      </geometry>
-      <material name="">
-        <color rgba="0.79216 0.81961 0.93333 1" />
-      </material>
-    </visual>
-    <collision>
-      <origin xyz="0 0 0" rpy="0 0 0" />
-      <geometry>
-        <mesh filename="package://probot_description/meshes/link_1.STL" />
+        <mesh filename="package://probot_description/meshes/PROBOT_Anno/link_1.STL" />
+      </geometry>
+      <material name="">
+        <color rgba="0.79216 0.81961 0.93333 1" />
+      </material>
+    </visual>
+    <collision>
+      <origin xyz="0 0 0" rpy="0 0 0" />
+      <geometry>
+        <mesh filename="package://probot_description/meshes/PROBOT_Anno/link_1.STL" />
       </geometry>
     </collision>
@@ -70,14 +70,14 @@
       <origin xyz="0 0 0" rpy="0 0 0" />
       <geometry>
-        <mesh filename="package://probot_description/meshes/link_2.STL" />
-      </geometry>
-      <material name="">
-        <color rgba="0.79216 0.81961 0.93333 1" />
-      </material>
-    </visual>
-    <collision>
-      <origin xyz="0 0 0" rpy="0 0 0" />
-      <geometry>
-        <mesh filename="package://probot_description/meshes/link_2.STL" />
+        <mesh filename="package://probot_description/meshes/PROBOT_Anno/link_2.STL" />
+      </geometry>
+      <material name="">
+        <color rgba="0.79216 0.81961 0.93333 1" />
+      </material>
+    </visual>
+    <collision>
+      <origin xyz="0 0 0" rpy="0 0 0" />
+      <geometry>
+        <mesh filename="package://probot_description/meshes/PROBOT_Anno/link_2.STL" />
       </geometry>
     </collision>
@@ -99,14 +99,14 @@
       <origin xyz="0 0 0" rpy="0 0 0" />
       <geometry>
-        <mesh filename="package://probot_description/meshes/link_3.STL" />
-      </geometry>
-      <material name="">
-        <color rgba="0.79216 0.81961 0.93333 1" />
-      </material>
-    </visual>
-    <collision>
-      <origin xyz="0 0 0" rpy="0 0 0" />
-      <geometry>
-        <mesh filename="package://probot_description/meshes/link_3.STL" />
+        <mesh filename="package://probot_description/meshes/PROBOT_Anno/link_3.STL" />
+      </geometry>
+      <material name="">
+        <color rgba="0.79216 0.81961 0.93333 1" />
+      </material>
+    </visual>
+    <collision>
+      <origin xyz="0 0 0" rpy="0 0 0" />
+      <geometry>
+        <mesh filename="package://probot_description/meshes/PROBOT_Anno/link_3.STL" />
       </geometry>
     </collision>
@@ -128,14 +128,14 @@
       <origin xyz="0 0 0" rpy="0 0 0" />
       <geometry>
-        <mesh filename="package://probot_description/meshes/link_4.STL" />
-      </geometry>
-      <material name="">
-        <color rgba="0.79216 0.81961 0.93333 1" />
-      </material>
-    </visual>
-    <collision>
-      <origin xyz="0 0 0" rpy="0 0 0" />
-      <geometry>
-        <mesh filename="package://probot_description/meshes/link_4.STL" />
+        <mesh filename="package://probot_description/meshes/PROBOT_Anno/link_4.STL" />
+      </geometry>
+      <material name="">
+        <color rgba="0.79216 0.81961 0.93333 1" />
+      </material>
+    </visual>
+    <collision>
+      <origin xyz="0 0 0" rpy="0 0 0" />
+      <geometry>
+        <mesh filename="package://probot_description/meshes/PROBOT_Anno/link_4.STL" />
       </geometry>
     </collision>
@@ -157,14 +157,14 @@
       <origin xyz="0 0 0" rpy="0 0 0" />
       <geometry>
-        <mesh filename="package://probot_description/meshes/link_5.STL" />
-      </geometry>
-      <material name="">
-        <color rgba="0.79216 0.81961 0.93333 1" />
-      </material>
-    </visual>
-    <collision>
-      <origin xyz="0 0 0" rpy="0 0 0" />
-      <geometry>
-        <mesh filename="package://probot_description/meshes/link_5.STL" />
+        <mesh filename="package://probot_description/meshes/PROBOT_Anno/link_5.STL" />
+      </geometry>
+      <material name="">
+        <color rgba="0.79216 0.81961 0.93333 1" />
+      </material>
+    </visual>
+    <collision>
+      <origin xyz="0 0 0" rpy="0 0 0" />
+      <geometry>
+        <mesh filename="package://probot_description/meshes/PROBOT_Anno/link_5.STL" />
       </geometry>
     </collision>
@@ -186,14 +186,14 @@
       <origin xyz="0 0 0" rpy="0 0 0" />
       <geometry>
-        <mesh filename="package://probot_description/meshes/link_6.STL" />
-      </geometry>
-      <material name="">
-        <color rgba="0.79216 0.81961 0.93333 1" />
-      </material>
-    </visual>
-    <collision>
-      <origin xyz="0 0 0" rpy="0 0 0" />
-      <geometry>
-        <mesh filename="package://probot_description/meshes/link_6.STL" />
+        <mesh filename="package://probot_description/meshes/PROBOT_Anno/link_6.STL" />
+      </geometry>
+      <material name="">
+        <color rgba="0.79216 0.81961 0.93333 1" />
+      </material>
+    </visual>
+    <collision>
+      <origin xyz="0 0 0" rpy="0 0 0" />
+      <geometry>
+        <mesh filename="package://probot_description/meshes/PROBOT_Anno/link_6.STL" />
       </geometry>
     </collision>

Commit message: Update robot software v2.1

File: probot_description/urdf/PROBOT_Anno/probot_anno.xacro (robot description, xacro)
@@ -2,10 +2,4 @@
 <robot name="probot_anno" xmlns:xacro="http://ros.org/wiki/xacro">
   <xacro:property name="M_PI" value="3.1415926536"/>
-  <link name="base_footprint"/>
-  <joint name="joint_0" type="fixed">
-    <origin xyz="0 0 0.02" rpy="0 0 0" />
-    <parent link="base_footprint" />
-    <child link="base_link" />
-  </joint>
   <link name="base_link">
     <inertial>
@@ -177,10 +171,10 @@
   <link name="link_6">
     <inertial>
-      <origin xyz="-0.010934 0.23134 0.0051509" rpy="0 0 0" />
-      <mass value="0.00001" />
-      <inertia ixx="10" ixy="0.0" ixz="0.0" iyy="10" iyz="0.0" izz="10" />
-    </inertial>
-    <visual>
-      <origin xyz="0 0 0" rpy="0 0 0" />
+      <origin xyz="-0.010934 0.23134 0.0051509" rpy="${-M_PI/2} 0 0" />
+      <mass value="0.00001" />
+      <inertia ixx="10" ixy="0.0" ixz="0.0" iyy="10" iyz="0.0" izz="10" />
+    </inertial>
+    <visual>
+      <origin xyz="0 0 0" rpy="${-M_PI/2} 0 0" />
       <geometry>
         <mesh filename="package://probot_description/meshes/PROBOT_Anno/link_6.STL" />
@@ -191,5 +185,5 @@
     </visual>
     <collision>
-      <origin xyz="0 0 0" rpy="0 0 0" />
+      <origin xyz="0 0 0" rpy="${-M_PI/2} 0 0" />
       <geometry>
         <mesh filename="package://probot_description/meshes/PROBOT_Anno/link_6.STL" />
@@ -198,13 +192,13 @@
   </link>
   <joint name="joint_6" type="revolute">
-    <origin xyz="0 -0.042 0" rpy="0 0 0" />
+    <origin xyz="0 -0.042 0" rpy="${M_PI/2} 0 0" />
     <parent link="link_5" />
     <child link="link_6" />
-    <axis xyz="0 -1 0" />
+    <axis xyz="0 0 1" />
     <limit lower="-3.1416" upper="3.1416" effort="100" velocity="3" />
   </joint>
   <link name="tool0"/>
   <joint name="joint_tool0" type="fixed">
-    <origin xyz="0 -0.013 0" rpy="${M_PI/2} 0 0" />
+    <origin xyz="0 0 0.013" rpy="${M_PI} 0 0" />
     <parent link="link_6" />
     <child link="tool0" />

File: probot_description/urdf/PROBOT_Anno/probot_anno_with_gripper.xacro (robot description, xacro)
@@ -4,10 +4,4 @@
   <xacro:include filename="$(find probot_description)/urdf/materials.urdf.xacro" />
   <xacro:include filename="$(find probot_description)/urdf/gripper.xacro" />
-  <link name="base_footprint"/>
-  <joint name="joint_0" type="fixed">
-    <origin xyz="0 0 0.02" rpy="0 0 0" />
-    <parent link="base_footprint" />
-    <child link="base_link" />
-  </joint>
   <link name="base_link">
     <inertial>
