Commit message: Fix robot model with gripper

File: probot_description/urdf/PROBOT_Anno/dynamixel_arm_hardware.xacro (robot description, xacro)
@@ -36,5 +36,5 @@
         <origin xyz=" 0 0 0 " rpy="0 0 0" />
         <geometry>
-          <mesh filename="package://probot_description/meshes/gripper/F10.stl" scale="${DYNAMIXEL_MESH_SCALE} ${DYNAMIXEL_MESH_SCALE} ${DYNAMIXEL_MESH_SCALE}"/>
+          <mesh filename="package://probot_description/meshes/PROBOT_Anno/gripper/F10.stl" scale="${DYNAMIXEL_MESH_SCALE} ${DYNAMIXEL_MESH_SCALE} ${DYNAMIXEL_MESH_SCALE}"/>
         </geometry>
         <material name="${color}"/>
@@ -67,5 +67,5 @@
         <origin xyz=" 0 0 0 " rpy="0 0 0" />
         <geometry>
-          <mesh filename="package://probot_description/meshes/gripper/F10.stl" scale="${DYNAMIXEL_MESH_SCALE} ${DYNAMIXEL_MESH_SCALE} ${DYNAMIXEL_MESH_SCALE}"/>
+          <mesh filename="package://probot_description/meshes/PROBOT_Anno/gripper/F10.stl" scale="${DYNAMIXEL_MESH_SCALE} ${DYNAMIXEL_MESH_SCALE} ${DYNAMIXEL_MESH_SCALE}"/>
         </geometry>
         <material name="${color}"/>
@@ -96,5 +96,5 @@
         <origin xyz=" 0 0 0 " rpy="0 0 0" />
         <geometry>
-          <mesh filename="package://probot_description/meshes/gripper/F2.stl" scale="${DYNAMIXEL_MESH_SCALE} ${DYNAMIXEL_MESH_SCALE} ${DYNAMIXEL_MESH_SCALE}"/>
+          <mesh filename="package://probot_description/meshes/PROBOT_Anno/gripper/F2.stl" scale="${DYNAMIXEL_MESH_SCALE} ${DYNAMIXEL_MESH_SCALE} ${DYNAMIXEL_MESH_SCALE}"/>
         </geometry>
         <material name="${color}"/>
@@ -125,5 +125,5 @@
         <origin xyz=" 0 0 0 " rpy="0 0 0" />
         <geometry>
-          <mesh filename="package://probot_description/meshes/gripper/finger.stl" scale="${DYNAMIXEL_MESH_SCALE} ${DYNAMIXEL_MESH_SCALE} ${DYNAMIXEL_MESH_SCALE}"/>
+          <mesh filename="package://probot_description/meshes/PROBOT_Anno/gripper/finger.stl" scale="${DYNAMIXEL_MESH_SCALE} ${DYNAMIXEL_MESH_SCALE} ${DYNAMIXEL_MESH_SCALE}"/>
         </geometry>
         <material name="${color}"/>
@@ -170,5 +170,5 @@
         <origin xyz=" 0 0 0 " rpy="0 0 0" />
         <geometry>
-          <mesh filename="package://probot_description/meshes/gripper/F3.stl" scale="${DYNAMIXEL_MESH_SCALE} ${DYNAMIXEL_MESH_SCALE} ${DYNAMIXEL_MESH_SCALE}"/>
+          <mesh filename="package://probot_description/meshes/PROBOT_Anno/gripper/F3.stl" scale="${DYNAMIXEL_MESH_SCALE} ${DYNAMIXEL_MESH_SCALE} ${DYNAMIXEL_MESH_SCALE}"/>
         </geometry>
         <material name="${color}"/>
@@ -199,5 +199,5 @@
         <origin xyz=" 0 0 0 " rpy="0 0 0" />
         <geometry>
-          <mesh filename="package://probot_description/meshes/gripper/F9.stl" scale="${DYNAMIXEL_MESH_SCALE} ${DYNAMIXEL_MESH_SCALE} ${DYNAMIXEL_MESH_SCALE}"/>
+          <mesh filename="package://probot_description/meshes/PROBOT_Anno/gripper/F9.stl" scale="${DYNAMIXEL_MESH_SCALE} ${DYNAMIXEL_MESH_SCALE} ${DYNAMIXEL_MESH_SCALE}"/>
         </geometry>
         <material name="${color}"/>
@@ -228,5 +228,5 @@
         <origin xyz=" 0 0 0 " rpy="0 0 0" />
         <geometry>
-          <mesh filename="package://probot_description/meshes/gripper/F11.stl" scale="${DYNAMIXEL_MESH_SCALE} ${DYNAMIXEL_MESH_SCALE} ${DYNAMIXEL_MESH_SCALE}"/>
+          <mesh filename="package://probot_description/meshes/PROBOT_Anno/gripper/F11.stl" scale="${DYNAMIXEL_MESH_SCALE} ${DYNAMIXEL_MESH_SCALE} ${DYNAMIXEL_MESH_SCALE}"/>
         </geometry>
         <material name="${color}"/>
@@ -257,5 +257,5 @@
         <origin xyz=" 0 0 0 " rpy="0 0 0" />
         <geometry>
-          <mesh filename="package://probot_description/meshes/gripper/ax12.${ARM_MESH_EXT}" scale="${DYNAMIXEL_MESH_SCALE} ${DYNAMIXEL_MESH_SCALE} ${DYNAMIXEL_MESH_SCALE}"/>
+          <mesh filename="package://probot_description/meshes/PROBOT_Anno/gripper/ax12.${ARM_MESH_EXT}" scale="${DYNAMIXEL_MESH_SCALE} ${DYNAMIXEL_MESH_SCALE} ${DYNAMIXEL_MESH_SCALE}"/>
         </geometry>
         <material name="Black"/>
@@ -288,5 +288,5 @@
         <origin xyz=" 0 0 0 " rpy="0 0 0" />
         <geometry>
-          <mesh filename="package://probot_description/meshes/gripper/ax12.${ARM_MESH_EXT}" scale="${DYNAMIXEL_MESH_SCALE} ${DYNAMIXEL_MESH_SCALE} ${DYNAMIXEL_MESH_SCALE}"/>
+          <mesh filename="package://probot_description/meshes/PROBOT_Anno/gripper/ax12.${ARM_MESH_EXT}" scale="${DYNAMIXEL_MESH_SCALE} ${DYNAMIXEL_MESH_SCALE} ${DYNAMIXEL_MESH_SCALE}"/>
         </geometry>
          <material name="Black"/>
@@ -319,5 +319,5 @@
         <origin xyz=" 0 0 0 " rpy="0 0 0" />
         <geometry>
-          <mesh filename="package://probot_description/meshes/gripper/F3.stl" scale="${DYNAMIXEL_MESH_SCALE} ${DYNAMIXEL_MESH_SCALE} ${DYNAMIXEL_MESH_SCALE}"/>
+          <mesh filename="package://probot_description/meshes/PROBOT_Anno/gripper/F3.stl" scale="${DYNAMIXEL_MESH_SCALE} ${DYNAMIXEL_MESH_SCALE} ${DYNAMIXEL_MESH_SCALE}"/>
         </geometry>
         <material name="${color}"/>
@@ -350,5 +350,5 @@
         <origin xyz=" 0 0 0 " rpy="0 0 0" />
         <geometry>
-          <mesh filename="package://probot_description/meshes/gripper/F2.stl" scale="${DYNAMIXEL_MESH_SCALE} ${DYNAMIXEL_MESH_SCALE} ${DYNAMIXEL_MESH_SCALE}"/>
+          <mesh filename="package://probot_description/meshes/PROBOT_Anno/gripper/F2.stl" scale="${DYNAMIXEL_MESH_SCALE} ${DYNAMIXEL_MESH_SCALE} ${DYNAMIXEL_MESH_SCALE}"/>
         </geometry>
         <material name="${color}"/>
@@ -381,5 +381,5 @@
         <origin xyz=" 0 0 0 " rpy="0 0 0" />
         <geometry>
-          <mesh filename="package://probot_description/meshes/gripper/F4.stl" scale="${DYNAMIXEL_MESH_SCALE} ${DYNAMIXEL_MESH_SCALE} ${DYNAMIXEL_MESH_SCALE}"/>
+          <mesh filename="package://probot_description/meshes/PROBOT_Anno/gripper/F4.stl" scale="${DYNAMIXEL_MESH_SCALE} ${DYNAMIXEL_MESH_SCALE} ${DYNAMIXEL_MESH_SCALE}"/>
         </geometry>
         <material name="${color}"/>

File: probot_description/urdf/PROBOT_Anno/gripper.xacro (robot description, xacro)
@@ -3,5 +3,5 @@
    <xacro:property name="PI" value="3.14159"/>
    <xacro:property name="DYNAMIXEL_MESH_SCALE" value="0.001"/>
-   <xacro:include filename="$(find probot_description)/urdf/dynamixel_arm_hardware.xacro" />
+   <xacro:include filename="$(find probot_description)/urdf/PROBOT_Anno/dynamixel_arm_hardware.xacro" />
    <xacro:macro name="gripper" params="parent color xyz rpy">
     <!-- gripper joint -->
@@ -28,5 +28,5 @@
         <origin xyz="0 0 0" rpy="0 0 0" />
         <geometry>
-          <mesh filename="package://probot_description/meshes/gripper/F2.stl" scale="${DYNAMIXEL_MESH_SCALE} ${DYNAMIXEL_MESH_SCALE} ${DYNAMIXEL_MESH_SCALE}"/>
+          <mesh filename="package://probot_description/meshes/PROBOT_Anno/gripper/F2.stl" scale="${DYNAMIXEL_MESH_SCALE} ${DYNAMIXEL_MESH_SCALE} ${DYNAMIXEL_MESH_SCALE}"/>
         </geometry>
         <material name="${color}"/>

File: probot_description/urdf/PROBOT_Anno/probot_anno_with_gripper.xacro (robot description, xacro)
@@ -2,6 +2,6 @@
 <robot name="probot_anno" xmlns:xacro="http://ros.org/wiki/xacro">
   <xacro:property name="M_PI" value="3.1415926536"/>
-  <xacro:include filename="$(find probot_description)/urdf/materials.urdf.xacro" />
-  <xacro:include filename="$(find probot_description)/urdf/gripper.xacro" />
+  <xacro:include filename="$(find probot_description)/urdf/PROBOT_Anno/materials.urdf.xacro" />
+  <xacro:include filename="$(find probot_description)/urdf/PROBOT_Anno/gripper.xacro" />
   <link name="base_link">
     <inertial>
@@ -228,5 +228,5 @@
   <xacro:transmission_block joint_name="joint_6"/>
   <xacro:transmission_block joint_name="gripper_finger_joint"/>
-  <xacro:include filename="$(find probot_description)/urdf/sensors/camera.urdf.xacro"/>
+  <xacro:include filename="$(find probot_description)/urdf/PROBOT_Anno/sensors/camera.urdf.xacro"/>
   <!-- ros_control plugin -->
   <gazebo>

File: probot_description/urdf/PROBOT_Anno/sensors/camera.urdf.xacro (robot description, xacro)
@@ -14,5 +14,5 @@
            <origin xyz="0 0 0" rpy="0 0 0"/>
            <geometry>
-           <mesh filename="package://probot_description/meshes/sensors/camera.STL" />
+           <mesh filename="package://probot_description/meshes/PROBOT_Anno/sensors/camera.STL" />
            </geometry>
        </collision>
@@ -20,5 +20,5 @@
            <origin xyz="0 0 0" rpy="${-M_PI} 0 ${-M_PI/2}"/>
            <geometry>
-           <mesh filename="package://probot_description/meshes/sensors/camera.STL" />
+           <mesh filename="package://probot_description/meshes/PROBOT_Anno/sensors/camera.STL" />
            </geometry>
            <material name="red"/>
@@ -32,4 +32,4 @@
        </inertial>
    </link>
-   <xacro:include filename="$(find probot_description)/urdf/sensors/camera.gazebo.xacro"/>
+   <xacro:include filename="$(find probot_description)/urdf/PROBOT_Anno/sensors/camera.gazebo.xacro"/>
 </robot>

Commit message: Update to V3.0.0

File: probot_description/urdf/PROBOT_Anno/dynamixel_arm_hardware.xacro (robot description, xacro)
@@ -47,4 +47,11 @@
       </collision>
     </link>
+        <gazebo reference="${name}_link">
+            <implicitSpringDamper>1</implicitSpringDamper>
+            <mu1>100000</mu1>
+            <mu2>100000</mu2>
+            <kp>100000000.0</kp>
+            <kd>1.0</kd>
+        </gazebo>
   </xacro:macro>
   <xacro:macro name="bioloid_F10_revolute" params="parent name color llimit ulimit vlimit *origin *axis">
@@ -78,4 +85,11 @@
       </collision>
     </link>
+        <gazebo reference="${name}_link">
+            <implicitSpringDamper>1</implicitSpringDamper>
+            <mu1>100000</mu1>
+            <mu2>100000</mu2>
+            <kp>100000000.0</kp>
+            <kd>1.0</kd>
+        </gazebo>
   </xacro:macro>
   <xacro:macro name="bioloid_F2_fixed" params="parent name color *origin">
@@ -107,4 +121,11 @@
       </collision>
     </link>
+        <gazebo reference="${name}_link">
+            <implicitSpringDamper>1</implicitSpringDamper>
+            <mu1>100000</mu1>
+            <mu2>100000</mu2>
+            <kp>100000000.0</kp>
+            <kd>1.0</kd>
+        </gazebo>
   </xacro:macro>
   <xacro:macro name="finger" params="parent name color *origin">
@@ -181,4 +202,11 @@
       </collision>
     </link>
+        <gazebo reference="${name}_link">
+            <implicitSpringDamper>1</implicitSpringDamper>
+            <mu1>100000</mu1>
+            <mu2>100000</mu2>
+            <kp>100000000.0</kp>
+            <kd>1.0</kd>
+        </gazebo>
   </xacro:macro>
   <xacro:macro name="bioloid_F9_fixed" params="parent name color *origin">
@@ -210,4 +238,11 @@
       </collision>
     </link>
+        <gazebo reference="${name}_link">
+            <implicitSpringDamper>1</implicitSpringDamper>
+            <mu1>100000</mu1>
+            <mu2>100000</mu2>
+            <kp>100000000.0</kp>
+            <kd>1.0</kd>
+        </gazebo>
   </xacro:macro>
   <xacro:macro name="bioloid_F11_fixed" params="parent name color *origin">
@@ -239,4 +274,11 @@
       </collision>
     </link>
+        <gazebo reference="${name}_link">
+            <implicitSpringDamper>1</implicitSpringDamper>
+            <mu1>100000</mu1>
+            <mu2>100000</mu2>
+            <kp>100000000.0</kp>
+            <kd>1.0</kd>
+        </gazebo>
   </xacro:macro>
   <xacro:macro name="dynamixel_AX12_fixed" params="parent name *origin">
@@ -268,4 +310,11 @@
       </collision>
     </link>
+        <gazebo reference="${name}_link">
+            <implicitSpringDamper>1</implicitSpringDamper>
+            <mu1>100000</mu1>
+            <mu2>100000</mu2>
+            <kp>100000000.0</kp>
+            <kd>1.0</kd>
+        </gazebo>
   </xacro:macro>
   <xacro:macro name="dynamixel_AX12_revolute" params="parent name llimit ulimit vlimit *origin *axis">
@@ -299,4 +348,11 @@
       </collision>
     </link>
+        <gazebo reference="${name}_link">
+            <implicitSpringDamper>1</implicitSpringDamper>
+            <mu1>100000</mu1>
+            <mu2>100000</mu2>
+            <kp>100000000.0</kp>
+            <kd>1.0</kd>
+        </gazebo>
   </xacro:macro>
   <xacro:macro name="bioloid_F3_revolute" params="parent name color llimit ulimit vlimit *origin *axis">
@@ -330,4 +386,11 @@
       </collision>
     </link>
+        <gazebo reference="${name}_link">
+            <implicitSpringDamper>1</implicitSpringDamper>
+            <mu1>100000</mu1>
+            <mu2>100000</mu2>
+            <kp>100000000.0</kp>
+            <kd>1.0</kd>
+        </gazebo>
   </xacro:macro>
   <xacro:macro name="bioloid_F2_revolute" params="parent name color llimit ulimit vlimit *origin *axis">
@@ -361,4 +424,11 @@
       </collision>
     </link>
+        <gazebo reference="${name}_link">
+            <implicitSpringDamper>1</implicitSpringDamper>
+            <mu1>100000</mu1>
+            <mu2>100000</mu2>
+            <kp>100000000.0</kp>
+            <kd>1.0</kd>
+        </gazebo>
   </xacro:macro>
   <xacro:macro name="bioloid_F4_revolute" params="parent name color llimit ulimit vlimit *origin *axis">
@@ -392,4 +462,11 @@
       </collision>
     </link>
+        <gazebo reference="${name}_link">
+            <implicitSpringDamper>1</implicitSpringDamper>
+            <mu1>100000</mu1>
+            <mu2>100000</mu2>
+            <kp>100000000.0</kp>
+            <kd>1.0</kd>
+        </gazebo>
   </xacro:macro>
 </robot>

File: probot_description/urdf/PROBOT_Anno/gripper.xacro (robot description, xacro)
@@ -76,4 +76,21 @@
       </inertial -->
     </link>
+    <gazebo>
+      <plugin name="gazebo_grasp_fix" filename="libgazebo_grasp_fix.so">
+            <arm>
+              <arm_name>robot</arm_name>
+              <palm_link>link_6</palm_link>
+              <gripper_link>gripper_active_finger_bracket_link</gripper_link>
+              <gripper_link>link_6</gripper_link>
+            </arm>
+        <forces_angle_tolerance>100</forces_angle_tolerance>
+        <update_rate>2</update_rate>
+        <grip_count_threshold>1</grip_count_threshold>
+        <max_grip_count>2</max_grip_count>
+        <release_tolerance>0.005</release_tolerance>
+        <disable_collisions_on_attach>true</disable_collisions_on_attach>
+        <contact_topic>__default_topic__</contact_topic>
+      </plugin>
+    </gazebo>
    </xacro:macro>
 </robot>

File: probot_description/urdf/PROBOT_Anno/probot_anno.xacro (robot description, xacro)
@@ -226,5 +226,5 @@
   <gazebo>
     <plugin name="gazebo_ros_control" filename="libgazebo_ros_control.so">
-      <robotNamespace>/probot_anno</robotNamespace>
+      <robotNamespace>/</robotNamespace>
       <robotSimType>gazebo_ros_control/DefaultRobotHWSim</robotSimType>
       <legacyModeNS>true</legacyModeNS>

File: probot_description/urdf/PROBOT_Anno/probot_anno_with_gripper.xacro (robot description, xacro)
@@ -4,8 +4,10 @@
   <xacro:include filename="$(find probot_description)/urdf/PROBOT_Anno/materials.urdf.xacro" />
   <xacro:include filename="$(find probot_description)/urdf/PROBOT_Anno/gripper.xacro" />
+  <xacro:include filename="$(find probot_description)/urdf/PROBOT_Anno/sensors/d435.urdf.xacro" />
+  <xacro:include filename="$(find probot_description)/urdf/PROBOT_Anno/sensors/realsense.gazebo.xacro"/>
   <link name="base_link">
     <inertial>
       <origin xyz="-0.010934 0.23134 0.0051509" rpy="0 0 0" />
-      <mass value="0.01" />
+      <mass value="0.8" />
       <inertia ixx="1.0" ixy="0.0" ixz="0.0" iyy="1.0" iyz="0.0" izz="1.0" />
     </inertial>
@@ -29,5 +31,5 @@
     <inertial>
       <origin xyz="-0.010934 0.23134 0.0051509" rpy="0 0 0" />
-      <mass value="0.01" />
+      <mass value="0.5" />
       <inertia ixx="1.0" ixy="0.0" ixz="0.0" iyy="1.0" iyz="0.0" izz="1.0" />
     </inertial>
@@ -228,9 +230,11 @@
   <xacro:transmission_block joint_name="joint_6"/>
   <xacro:transmission_block joint_name="gripper_finger_joint"/>
-  <xacro:include filename="$(find probot_description)/urdf/PROBOT_Anno/sensors/camera.urdf.xacro"/>
+  <sensor_d435 parent="base_link">
+    <origin xyz="0.3 0 0.7" rpy="0 ${M_PI/2} 0"/>
+  </sensor_d435>
   <!-- ros_control plugin -->
   <gazebo>
     <plugin name="gazebo_ros_control" filename="libgazebo_ros_control.so">
-      <robotNamespace>/probot_anno</robotNamespace>
+      <robotNamespace>/</robotNamespace>
       <robotSimType>gazebo_ros_control/DefaultRobotHWSim</robotSimType>
       <legacyModeNS>true</legacyModeNS>
